File: Non-Isolated/Modular-I2C-4PxRJ45-Relay-Driver.kicad_sch (KiCad schematic)
At the start: 123 parts, among them J1 Conn_02x03_Odd_Even, J2 Conn_02x03_Odd_Even, J3 Screw_Terminal_01x02, J4 Screw_Terminal_01x02, Q51 2N7002, Q52 2N7002, Q53 2N7002, Q54 2N7002, Q55 2N7002, Q56 2N7002, Q57 2N7002, Q58 2N7002, Q59 2N7002, Q60 2N7002, Q61 2N7002, Q62 2N7002, Q63 2N7002, Q64 2N7002, Q65 2N7002, Q66 2N7002, SW1 SW_DIP_x04, SW5 2P_DIP, U1 MCP23017_SO, U2 AP63205WU, U3 ELQ3H7(TA), U4 Conn_02x08_Row_Letter_First, U5 Conn_02x08_Row_Letter_First, U6 Conn_02x08_Row_Letter_First

Commit message: isolated
Parts:
- removed C6: 100nF, Capacitor_SMD:C_0603_1608Metric, symbol Device:C
- removed C7, C8: 22uF, Capacitor_SMD:C_0603_1608Metric, symbol Device:C
- removed C9: 10uF, Capacitor_SMD:C_0603_1608Metric, symbol Device:C
- removed D2: red, LED_SMD:LED_0603_1608Metric, symbol Device:LED
- removed L1: 4.7uH 3A, Inductor_SMD:L_6.3x6.3_H3, symbol pspice:INDUCTOR
- removed R1: 4.7k, Resistor_SMD:R_0603_1608Metric, symbol Device:R_US
- removed U2: AP63205WU, Package_TO_SOT_SMD:TSOT-23-6, symbol Regulator_Switching:AP63205WU
- removed U3: ELQ3H7(TA), Package_SO:SO-16_5.3x10.2mm_P1.27mm, symbol Connector_Generic_Shielded:Conn_02x08_Counter_Clockwise_Shielded
- removed U4, U5, U6: Conn_02x08_Row_Letter_First, Package_SO:SO-16_5.3x10.2mm_P1.27mm, symbol Connector_Generic_Shielded:Conn_02x08_Counter_Clockwise_Shielded
- R51, R52, R53, R54, R55, R56, R57, R58, R59, R60, R61, R62, R63, R64, R65, R66: value 10K -> 1K; LCSC C25804 -> C21190
Connections:
- net GNDPWR is gone; now on net GNDREF: C5.2, J3.2, J4.2, Q51.3 (S), Q52.3 (S), Q53.3 (S), Q54.3 (S), Q55.3 (S), Q56.3 (S), Q57.3 (S), Q58.3 (S), Q59.3 (S), Q60.3 (S), Q61.3 (S), Q62.3 (S), Q63.3 (S), Q64.3 (S), Q65.3 (S), Q66.3 (S), R5.2, RJ45-1.EH
- net p1-a5 is gone; now on net p1-a: Q51.2 (G)
- net p1-b5 is gone; now on net p1-b: Q52.2 (G)
- net p1-c5 is gone; now on net p1-c: Q53.2 (G)
- net p1-d5 is gone; now on net p1-d: Q54.2 (G)
- net p2-a5 is gone; now on net p2-a: Q55.2 (G)
- net p2-b5 is gone; now on net p2-b: Q56.2 (G)
- net p2-c5 is gone; now on net p2-c: Q57.2 (G)
- net p2-d5 is gone; now on net p2-d: Q58.2 (G)
- net p3-a5 is gone; now on net p3-a: Q59.2 (G)
- net p3-b5 is gone; now on net p3-b: Q60.2 (G)
- net p3-c5 is gone; now on net p3-c: Q61.2 (G)
- net p3-d5 is gone; now on net p3-d: Q62.2 (G)
- net p4-a5 is gone; now on net p4-a: Q63.2 (G)
- net p4-b5 is gone; now on net p4-b: Q64.2 (G)
- net p4-c5 is gone; now on net p4-c: Q65.2 (G)
- net p4-d5 is gone; now on net p4-d: Q66.2 (G)
Other:
- moved on the sheet: C5, D3, D4, D51, D52, D53, D54, D55, D56, D57, D58, D59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
