File: Modular-I2C-4PxRJ45-Relay-Driver.kicad_sch (KiCad schematic)
At the start: 123 parts, among them J1 Conn_02x03_Odd_Even, J2 Conn_02x03_Odd_Even, J3 Screw_Terminal_01x02, J4 Screw_Terminal_01x02, Q51 2N7002, Q52 2N7002, Q53 2N7002, Q54 2N7002, Q55 2N7002, Q56 2N7002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

Commit message: optocoupler update
Parts:
- U3: LCSC C89878 -> C146217
- U4, U5, U6: value Conn_02x08_Row_Letter_First -> ELQ3H7(TA); LCSC C89878 -> C146217
Changed lines of the file:
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@@
     (pin "2")
   )
+  (symbol (lib_name "Conn_02x08_Counter_Clockwise_Shielded_1") (lib_id "Connector_Generic_Shielded:Conn_02x08_Counter_Clockwise_Shielded") (at 96.52 -182.88 0) (unit 1)
+    (in_bom yes) (on_board yes)
+    (property "Reference" "U4" (id 0) (at 97.79 -195.58 0)
+      (effects (font (size 1.27 1.27)) hide)
+    )
+    (property "Value" "ELQ3H7(TA)" (id 1) (at 97.79 -195.58 0))
+    (property "Footprint" "Package_SO:SO-16_5.3x10.2mm_P1.27mm" (id 2) (at 99.06 -170.18 0)
+      (effects (font (size 1.27 1.27)) hide)
+    )
+    (property "Datasheet" "~" (id 3) (at 96.52 -182.88 0)
+      (effects (font (size 1.27 1.27)) hide)
+    )
+    (property "LCSC" "C146217" (id 4) (at 97.79 -193.04 0)
+      (effects (font (size 1 1)))
+    )
+    (pin "1")
+    (pin "10")
+    (pin "11")
+    (pin "12")
+    (pin "13")
+    (pin "14")
+    (pin "15")
+    (pin "16")
+    (pin "2")
+    (pin "3")
+    (pin "4")
+    (pin "5")
+    (pin "6")
+    (pin "7")
+    (pin "8")
+    (pin "9")
+  )
   (symbol (lib_id "power:GNDREF") (at -270.51 179.07 0) (unit 1)
     (in_bom yes) (on_board yes) (fields_autoplaced)
@@
     (pin "1")
   )
-  (symbol (lib_id "Connector_Generic_Shielded:Conn_02x08_Counter_Clockwise_Shielded") (at -109.22 7.62 0) (unit 1)
+  (symbol (lib_name "Conn_02x08_Counter_Clockwise_Shielded_1") (lib_id "Connector_Generic_Shielded:Conn_02x08_Counter_Clockwise_Shielded") (at -109.22 7.62 0) (unit 1)
     (in_bom yes) (on_board yes)
     (property "Reference" "U3" (id 0) (at -107.95 -5.08 0)
@@
     )
     (property "Value" "ELQ3H7(TA)" (id 1) (at -107.95 -5.08 0))
-    (property "Footprint" "Package_SO:SO-16_5.3x10.2mm_P1.27mm" (id 2) (at -109.22 7.62 0)
+    (property "Footprint" "Package_SO:SO-16_5.3x10.2mm_P1.27mm" (id 2) (at -106.68 20.32 0)
       (effects (font (size 1.27 1.27)) hide)
     )
@@
       (effects (font (size 1.27 1.27)) hide)
     )
-    (property "LCSC" "C89878" (id 4) (at -107.95 -2.54 0)
+    (property "LCSC" "C146217" (id 4) (at -107.95 -2.54 0)
       (effects (font (size 1 1)))
     )
@@
     (pin "8")
     (pin "9")
-    (pin "SH")
   )
   (symbol (lib_id "power:GNDREF") (at 59.69 -182.88 0) (unit 1)
@@
     (pin "3")
   )
+  (symbol (lib_name "Conn_02x08_Counter_Clockwise_Shielded_1") (lib_id "Connector_Generic_Shielded:Conn_02x08_Counter_Clockwise_Shielded") (at 229.87 -185.42 0) (unit 1)
+    (in_bom yes) (on_board yes)
+    (property "Reference" "U5" (id 0) (at 231.14 -198.12 0)
+      (effects (font (size 1.27 1.27)) hide)
+    )
+    (property "Value" "ELQ3H7(TA)" (id 1) (at 231.14 -198.12 0))
+    (property "Footprint" "Package_SO:SO-16_5.3x10.2mm_P1.27mm" (id 2) (at 232.41 -172.72 0)
+      (effects (font (size 1.27 1.27)) hide)
+    )
+    (property "Datasheet" "~" (id 3) (at 229.87 -185.42 0)
+      (effects (font (size 1.27 1.27)) hide)
+    )
+    (property "LCSC" "C146217" (id 4) (at 231.14 -195.58 0)
+      (effects (font (size 1 1)))
+    )
+    (pin "1")
+    (pin "10")
+    (pin "11")
+    (pin "12")
+    (pin "13")
+    (pin "14")
+    (pin "15")
+    (pin "16")
+    (pin "2")
+    (pin "3")
+    (pin "4")
+    (pin "5")
+    (pin "6")
+    (pin "7")
+    (pin "8")
+    (pin "9")
+  )
   (symbol (lib_id "LED:IR26-21C_L110_TR8") (at 71.12 -110.49 180) (unit 1)
     (in_bom yes) (on_board yes)
@@
     (pin "1")
   )
-  (symbol (lib_id "Connector_Generic_Shielded:Conn_02x08_Counter_Clockwise_Shielded") (at 96.52 -182.88 0) (unit 1)
-    (in_bom yes) (on_board yes) (fields_autoplaced)
-    (property "Reference" "U4" (id 0) (at 97.79 -195.58 0))
-    (property "Value" "Conn_02x08_Row_Letter_First" (id 1) (at 97.79 -193.04 0))
-    (property "Footprint" "Package_SO:SO-16_5.3x10.2mm_P1.27mm" (id 2) (at 96.52 -182.88 0)
-      (effects (font (size 1.27 1.27)) hide)
-    )
-    (property "Datasheet" "~" (id 3) (at 96.52 -182.88 0)
-      (effects (font (size 1.27 1.27)) hide)
-    )
-    (property "LCSC" "C89878" (id 4) (at 96.52 -182.88 0)
-      (effects (font (size 1 1)) hide)
-    )
-    (pin "1")
-    (pin "10")
-    (pin "11")
-    (pin "12")
-    (pin "13")
-    (pin "14")
-    (pin "15")
-    (pin "16")
-    (pin "2")
-    (pin "3")
-    (pin "4")
-    (pin "5")
-    (pin "6")
-    (pin "7")
-    (pin "8")
-    (pin "9")
-    (pin "SH")
-  )
   (symbol (lib_id "Device:R") (at -127 48.26 270) (mirror x) (unit 1)
     (in_bom yes) (on_board yes)
@@
     (pin "8")
   )
+  (symbol (lib_name "Conn_02x08_Counter_Clockwise_Shielded_1") (lib_id "Connector_Generic_Shielded:Conn_02x08_Counter_Clockwise_Shielded") (at 360.68 -185.42 0) (unit 1)
+    (in_bom yes) (on_board yes)
+    (property "Reference" "U6" (id 0) (at 361.95 -198.12 0)
+      (effects (font (size 1.27 1.27)) hide)
+    )
+    (property "Value" "ELQ3H7(TA)" (id 1) (at 361.95 -198.12 0))
+    (property "Footprint" "Package_SO:SO-16_5.3x10.2mm_P1.27mm" (id 2) (at 363.22 -172.72 0)
+      (effects (font (size 1.27 1.27)) hide)
+    )
+    (property "Datasheet" "~" (id 3) (at 360.68 -185.42 0)
+      (effects (font (size 1.27 1.27)) hide)
+    )
+    (property "LCSC" "C146217" (id 4) (at 361.95 -195.58 0)
+      (effects (font (size 1 1)))
+    )
+    (pin "1")
+    (pin "10")
+    (pin "11")
+    (pin "12")
+    (pin "13")
+    (pin "14")
+    (pin "15")
+    (pin "16")
+    (pin "2")
+    (pin "3")
+    (pin "4")
+    (pin "5")
+    (pin "6")
+    (pin "7")
+    (pin "8")
+    (pin "9")
+  )
   (symbol (lib_id "Device:R") (at 81.28 -138.43 270) (mirror x) (unit 1)
     (in_bom yes) (on_board yes)
@@
     (pin "1")
   )
-  (symbol (lib_id "Connector_Generic_Shielded:Conn_02x08_Counter_Clockwise_Shielded") (at 229.87 -185.42 0) (unit 1)
-    (in_bom yes) (on_board yes) (fields_autoplaced)
-    (property "Reference" "U5" (id 0) (at 231.14 -198.12 0))
-    (property "Value" "Conn_02x08_Row_Letter_First" (id 1) (at 231.14 -195.58 0))
-    (property "Footprint" "Package_SO:SO-16_5.3x10.2mm_P1.27mm" (id 2) (at 229.87 -185.42 0)
-      (effects (font (size 1.27 1.27)) hide)
-    )
-    (property "Datasheet" "~" (id 3) (at 229.87 -185.42 0)
-      (effects (font (size 1.27 1.27)) hide)
-    )
-    (property "LCSC" "C89878" (id 4) (at 229.87 -185.42 0)
-      (effects (font (size 1 1)) hide)
-    )
-    (pin "1")
-    (pin "10")
-    (pin "11")
-    (pin "12")
-    (pin "13")
-    (pin "14")
-    (pin "15")
-    (pin "16")
-    (pin "2")
-    (pin "3")
-    (pin "4")
-    (pin "5")
-    (pin "6")
-    (pin "7")
-    (pin "8")
-    (pin "9")
-    (pin "SH")
-  )
   (symbol (lib_id "LED:IR26-21C_L110_TR8") (at 332.74 -82.55 180) (unit 1)
     (in_bom yes) (on_board yes)
@@
     (pin "8")
   )
-  (symbol (lib_id "Connector_Generic_Shielded:Conn_02x08_Counter_Clockwise_Shielded") (at 360.68 -185.42 0) (unit 1)
-    (in_bom yes) (on_board yes) (fields_autoplaced)
-    (property "Reference" "U6" (id 0) (at 361.95 -198.12 0))
-    (property "Value" "Conn_02x08_Row_Letter_First" (id 1) (at 361.95 -195.58 0))
-    (property "Footprint" "Package_SO:SO-16_5.3x10.2mm_P1.27mm" (id 2) (at 360.68 -185.42 0)
-      (effects (font (size 1.27 1.27)) hide)
-    )
-    (property "Datasheet" "~" (id 3) (at 360.68 -185.42 0)
-      (effects (font (size 1.27 1.27)) hide)
-    )
-    (property "LCSC" "C89878" (id 4) (at 360.68 -185.42 0)
-      (effects (font (size 1 1)) hide)
-    )
-    (pin "1")
-    (pin "10")
-    (pin "11")
-    (pin "12")
-    (pin "13")
-    (pin "14")
-    (pin "15")
-    (pin "16")
-    (pin "2")
-    (pin "3")
-    (pin "4")
-    (pin "5")
-    (pin "6")
-    (pin "7")
-    (pin "8")
-    (pin "9")
-    (pin "SH")
-  )
   (symbol (lib_id "power:GNDPWR") (at -115.57 60.96 0) (unit 1)
     (in_bom yes) (on_board yes) (fields_autoplaced)
@@
       (reference "U3") (unit 1) (value "ELQ3H7(TA)") (footprint "Package_SO:SO-16_5.3x10.2mm_P1.27mm")
     )
-    (path "/80e1febd-db3d-40c9-a0b4-7e2be5196af1"
-      (reference "U4") (unit 1) (value "Conn_02x08_Row_Letter_First") (footprint "Package_SO:SO-16_5.3x10.2mm_P1.27mm")
+    (path "/0e8c37d9-5317-4290-a93b-bf9c54910b5f"
+      (reference "U4") (unit 1) (value "ELQ3H7(TA)") (footprint "Package_SO:SO-16_5.3x10.2mm_P1.27mm")
     )
-    (path "/c70c1291-92bd-48d8-9851-68847b1aa846"
-      (reference "U5") (unit 1) (value "Conn_02x08_Row_Letter_First") (footprint "Package_SO:SO-16_5.3x10.2mm_P1.27mm")
+    (path "/79c8b881-10b9-4fc2-af42-e8f638ba0ce2"
+      (reference "U5") (unit 1) (value "ELQ3H7(TA)") (footprint "Package_SO:SO-16_5.3x10.2mm_P1.27mm")
     )
-    (path "/cdc52a2e-7e16-46dd-8286-9c88e243aed0"
-      (reference "U6") (unit 1) (value "Conn_02x08_Row_Letter_First") (footprint "Package_SO:SO-16_5.3x10.2mm_P1.27mm")
+    (path "/b860eb85-80ab-4fb4-a4fc-c95aeac18412"
+      (reference "U6") (unit 1) (value "ELQ3H7(TA)") (footprint "Package_SO:SO-16_5.3x10.2mm_P1.27mm")
     )
   )

Commit message: added 3d models
Parts:
- J3, J4: footprint Austins creations:2pinblock -> Vizista:CONN-TH_WJ2EDGVC-5.08-2P
Changed lines of the file:
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@@
       (effects (font (size 1.27 1.27)) (justify right))
     )
-    (property "Footprint" "Austins creations:2pinblock" (id 2) (at -278.13 129.54 0)
+    (property "Footprint" "Vizista:CONN-TH_WJ2EDGVC-5.08-2P" (id 2) (at -278.13 129.54 0)
       (effects (font (size 1.27 1.27)) hide)
     )
@@
       (effects (font (size 1.27 1.27)) (justify right))
     )
-    (property "Footprint" "Austins creations:2pinblock" (id 2) (at -278.13 114.3 0)
+    (property "Footprint" "Vizista:CONN-TH_WJ2EDGVC-5.08-2P" (id 2) (at -278.13 114.3 0)
       (effects (font (size 1.27 1.27)) hide)
     )
@@
     )
     (path "/5c80bb60-c1a7-4555-aac8-f98784916264"
-      (reference "J3") (unit 1) (value "Screw_Terminal_01x02") (footprint "Austins creations:2pinblock")
+      (reference "J3") (unit 1) (value "Screw_Terminal_01x02") (footprint "Vizista:CONN-TH_WJ2EDGVC-5.08-2P")
     )
     (path "/2e2f44e0-bff2-476d-8545-70d22caf66d0"
-      (reference "J4") (unit 1) (value "Screw_Terminal_01x02") (footprint "Austins creations:2pinblock")
+      (reference "J4") (unit 1) (value "Screw_Terminal_01x02") (footprint "Vizista:CONN-TH_WJ2EDGVC-5.08-2P")
     )
     (path "/f1a83b46-a1ba-46e2-99b0-69508149769e"

Commit message: 3d update, manufacturing files
Parts:
- R3: LCSC C25804 -> C25804
- RJ45-1: LCSC (none) -> C77852; part # C77852 -> (none)
- SW5: LCSC C2758181 -> C976364
Changed lines of the file:
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@@
       (effects (font (size 1.27 1.27)) hide)
     )
-    (property "LCSC" "C25804 " (id 4) (at -215.9 135.89 90)
+    (property "LCSC" "C25804" (id 4) (at -215.9 135.89 90)
       (effects (font (size 1 1)))
     )
@@
       (effects (font (size 1.27 1.27)) hide)
     )
-    (property "LCSC" "C2758181" (id 4) (at -229.87 139.7 0))
+    (property "LCSC" "C976364" (id 4) (at -229.87 139.7 0))
     (pin "1")
     (pin "2")
@@
       (effects (font (size 1.27 1.27)) hide)
     )
-    (property "part #" "C77852" (id 4) (at -16.51 34.29 0)
-      (effects (font (size 1 1)))
-    )
+    (property "LCSC" "C77852" (id 4) (at -16.51 34.29 0)
+      (effects (font (size 1 1)))
+    )
