File: Modular-I2C-4PxRJ45-Relay-Driver.kicad_pcb (KiCad board)
At the start: 2 copper layers, 69.5 x 100 mm, 111 parts, among them J1 Conn_02x03_Odd_Even, J2 Conn_02x03_Odd_Even, J3 Screw_Terminal_01x02, J4 Screw_Terminal_01x02, Q51 2N7002, Q52 2N7002, Q53 2N7002, Q54 2N7002, Q55 2N7002, Q56 2N7002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

Commit message: isolated
Parts:
- added C6: 100nF, Capacitor_SMD:C_0603_1608Metric, F.Cu at (127.4, 78.2)
- added C7: 22uF, Capacitor_SMD:C_0603_1608Metric, F.Cu at (123.5, 79.8)
- added C8: 22uF, Capacitor_SMD:C_0603_1608Metric, F.Cu at (123.4, 82.5)
- added C9: 10uF, Capacitor_SMD:C_0603_1608Metric, F.Cu at (130.7, 81.1)
- added D2: red, LED_SMD:LED_0603_1608Metric, F.Cu at (118.7, 79.0)
- added L1: 4.7uH 3A, Inductor_SMD:L_6.3x6.3_H3, F.Cu at (127.1, 73.0)
- added R1: 4.7k, Resistor_SMD:R_0603_1608Metric, F.Cu at (118.6, 76.3)
- added U2: AP63205WU, Package_TO_SOT_SMD:TSOT-23-6, F.Cu at (127.3, 81.4)
- added U3: ELQ3H7(TA), Package_SO:SO-16_5.3x10.2mm_P1.27mm, F.Cu at (131.7, 61.0)
- added U4: Conn_02x08_Row_Letter_First, Package_SO:SO-16_5.3x10.2mm_P1.27mm, F.Cu at (143.5, 61.0)
- added U5: Conn_02x08_Row_Letter_First, Package_SO:SO-16_5.3x10.2mm_P1.27mm, F.Cu at (155.2, 61.0)
- added U6: Conn_02x08_Row_Letter_First, Package_SO:SO-16_5.3x10.2mm_P1.27mm, F.Cu at (166.5, 61.0)
- R51, R52, R53, R54, R55, R56, R57, R58, R59, R60, R61, R62, R63, R64, R65, R66: value 1K -> 10K
- moved J3 47.9 mm to (139.3, 73.7)
- moved J4 47.9 mm to (165.8, 73.7)
- moved C5 47.9 mm to (152.5, 76.8)
- moved D3 39.2 mm to (173.9, 74.2)
- moved R5 39.2 mm to (176.7, 75.0)
- moved R6 21.1 mm to (178.4, 40.8)
- moved D4 20.3 mm to (175.9, 41.3)
- moved J2 19.0 mm to (121.8, 54.9)
- moved J1 18.9 mm to (179.1, 55.0)
- moved RN5 17.9 mm to (158.1, 37.7)
- moved RN3 17.9 mm to (158.1, 42.2)
- moved D8 17.8 mm to (129.4, 51.1)
- moved C3 17.5 mm to (151.8, 32.6)
- moved U1 16.4 mm to (141.6, 35.7)
- moved RN15 16.3 mm to (149.5, 37.6)
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Connections:
- C5 pad 2: GNDREF -> GNDPWR
- J3 pad 2: GNDREF -> GNDPWR
- J4 pad 2: GNDREF -> GNDPWR
- Q51 pad 2: p1-a -> p1-a5
- Q51 pad 3: GNDREF -> GNDPWR
- Q52 pad 2: p1-b -> p1-b5
- Q52 pad 3: GNDREF -> GNDPWR
- Q53 pad 2: p1-c -> p1-c5
- Q53 pad 3: GNDREF -> GNDPWR
- Q54 pad 2: p1-d -> p1-d5
- Q54 pad 3: GNDREF -> GNDPWR
- Q55 pad 2: p2-a -> p2-a5
- Q55 pad 3: GNDREF -> GNDPWR
- Q56 pad 2: p2-b -> p2-b5
- Q56 pad 3: GNDREF -> GNDPWR
- Q57 pad 2: p2-c -> p2-c5
- Q57 pad 3: GNDREF -> GNDPWR
- Q58 pad 2: p2-d -> p2-d5
- Q58 pad 3: GNDREF -> GNDPWR
- Q59 pad 2: p3-a -> p3-a5
- Q59 pad 3: GNDREF -> GNDPWR
- Q60 pad 2: p3-b -> p3-b5
- Q60 pad 3: GNDREF -> GNDPWR
- Q61 pad 2: p3-c -> p3-c5
- Q61 pad 3: GNDREF -> GNDPWR
- Q62 pad 2: p3-d -> p3-d5
- Q62 pad 3: GNDREF -> GNDPWR
- Q63 pad 2: p4-a -> p4-a5
- Q63 pad 3: GNDREF -> GNDPWR
- Q64 pad 2: p4-b -> p4-b5
- Q64 pad 3: GNDREF -> GNDPWR
- Q65 pad 2: p4-c -> p4-c5
- Q65 pad 3: GNDREF -> GNDPWR
- Q66 pad 2: p4-d -> p4-d5
- Q66 pad 3: GNDREF -> GNDPWR
- R5 pad 2: GNDREF -> GNDPWR
- RJ45-1 pad EH: GNDREF -> GNDPWR
Routing:
- net +5V: track 0.00 -> 121.4 mm
- net VCC: track 145.9 -> 182.3 mm
- net p4-d5: track 0.00 -> 32.5 mm, vias 0 -> 2
- net p1-a5: track 0.00 -> 32.3 mm, vias 0 -> 2
- net p4-c5: track 0.00 -> 31.7 mm, vias 0 -> 2
- net p1-b5: track 0.00 -> 31.6 mm, vias 0 -> 2
- net p4-b5: track 0.00 -> 31.1 mm, vias 0 -> 2
- net p1-c5: track 0.00 -> 30.9 mm, vias 0 -> 2
- net p2-a5: track 0.00 -> 30.4 mm, vias 0 -> 2
- net p4-a5: track 0.00 -> 30.3 mm, vias 0 -> 2
- net p1-d5: track 0.00 -> 30.3 mm, vias 0 -> 2
- net p3-d5: track 0.00 -> 29.9 mm, vias 0 -> 2
- net p2-b5: track 0.00 -> 29.5 mm, vias 0 -> 2
- net p3-c5: track 0.00 -> 29.2 mm, vias 0 -> 2
- net VDD: track 327.6 -> 298.8 mm
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- added copper zone on B.Cu, net GNDPWR
- added copper zone on F.Cu, net GNDPWR
Other:
- outline, holes or cut-outs redrawn
- board text added: "+"
- board text added: "-"
- board text added: "A 1 2 3 4 5 6 7 8"
- board text added: "Based on design by Jon Oxer by Austin's Creations modified by Mattar"
- board text removed: "Modular 4-Port I2CRJ45 Relay Driver Breakout"
- board text removed: "by Jon Oxer Modified By Austin's Creations"

Commit message: optocoupler update
Parts:
- U4, U5, U6: value Conn_02x08_Row_Letter_First -> ELQ3H7(TA)
Routing:
- net VDD: track 298.8 -> 300.9 mm
Changed lines of the file:
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@@
   (net 104 "unconnected-(D8-Pad6)")
   (net 105 "GNDPWR")
-  (net 106 "Net-(U2-Pad5)")
-  (net 107 "Net-(U2-Pad6)")
+  (net 106 "Net-(C6-Pad1)")
+  (net 107 "Net-(C6-Pad2)")
   (net 108 "+5V")
   (net 109 "p1-a5")
@@
     (descr "SO, 16 Pin (https://www.ti.com/lit/ml/msop002a/msop002a.pdf), generated with kicad-footprint-generator ipc_gullwing_generator.py")
     (tags "SO SO")
-    (property "LCSC" "C89878")
+    (property "LCSC" "C146217")
     (property "Sheetfile" "Modular-I2C-4PxRJ45-Relay-Driver.kicad_sch")
     (property "Sheetname" "")
@@
       (effects (font (size 1 1) (thickness 0.15)))
     )
-    (fp_text value "Conn_02x08_Row_Letter_First" (at 0 6.05 90) (layer "F.Fab") hide
+    (fp_text value "ELQ3H7(TA)" (at 0 6.05 90) (layer "F.Fab") hide
       (effects (font (size 1 1) (thickness 0.15)))
     )
@@
     (descr "SO, 16 Pin (https://www.ti.com/lit/ml/msop002a/msop002a.pdf), generated with kicad-footprint-generator ipc_gullwing_generator.py")
     (tags "SO SO")
-    (property "LCSC" "C89878")
+    (property "LCSC" "C146217")
     (property "Sheetfile" "Modular-I2C-4PxRJ45-Relay-Driver.kicad_sch")
     (property "Sheetname" "")
@@
       (effects (font (size 1 1) (thickness 0.15)))
     )
-    (fp_text value "Conn_02x08_Row_Letter_First" (at 0 6.05 90) (layer "F.Fab") hide
+    (fp_text value "ELQ3H7(TA)" (at 0 6.05 90) (layer "F.Fab") hide
       (effects (font (size 1 1) (thickness 0.15)))
     )
@@
       (net 105 "GNDPWR") (pinfunction "GND") (pintype "power_in"))
     (pad "5" smd roundrect (at 1.1375 0 90) (size 1.325 0.6) (layers "F.Cu" "F.Paste" "F.Mask") (roundrect_rratio 0.25)
-      (net 106 "Net-(U2-Pad5)") (pinfunction "SW") (pintype "output"))
+      (net 106 "Net-(C6-Pad1)") (pinfunction "SW") (pintype "output"))
     (pad "6" smd roundrect (at 1.1375 -0.95 90) (size 1.325 0.6) (layers "F.Cu" "F.Paste" "F.Mask") (roundrect_rratio 0.25)
-      (net 107 "Net-(U2-Pad6)") (pinfunction "BST") (pintype "passive"))
+      (net 107 "Net-(C6-Pad2)") (pinfunction "BST") (pintype "passive"))
     (model "${KICAD6_3DMODEL_DIR}/Package_TO_SOT_SMD.3dshapes/TSOT-23-6.wrl"
       (offset (xyz 0 0 0))
@@
     (descr "SO, 16 Pin (https://www.ti.com/lit/ml/msop002a/msop002a.pdf), generated with kicad-footprint-generator ipc_gullwing_generator.py")
     (tags "SO SO")
-    (property "LCSC" "C89878")
+    (property "LCSC" "C146217")
     (property "Sheetfile" "Modular-I2C-4PxRJ45-Relay-Driver.kicad_sch")
     (property "Sheetname" "")
@@
     (fp_arc (start 1.91 1.91) (mid 0 2.701148) (end -1.91 1.91) (layer "F.Fab") (width 0.1))
     (pad "1" smd rect (at -2.75 0 180) (size 1.5 2.4) (layers "F.Cu" "F.Paste" "F.Mask")
-      (net 106 "Net-(U2-Pad5)") (pinfunction "1") (pintype "input"))
+      (net 106 "Net-(C6-Pad1)") (pinfunction "1") (pintype "input"))
     (pad "2" smd rect (at 2.75 0 180) (size 1.5 2.4) (layers "F.Cu" "F.Paste" "F.Mask")
       (net 108 "+5V") (pinfunction "2") (pintype "input"))
@@
     (descr "SO, 16 Pin (https://www.ti.com/lit/ml/msop002a/msop002a.pdf), generated with kicad-footprint-generator ipc_gullwing_generator.py")
     (tags "SO SO")
-    (property "LCSC" "C89878")
+    (property "LCSC" "C146217")
     (property "Sheetfile" "Modular-I2C-4PxRJ45-Relay-Driver.kicad_sch")
     (property "Sheetname" "")
@@
       (effects (font (size 1 1) (thickness 0.15)))
     )
-    (fp_text value "Conn_02x08_Row_Letter_First" (at 0 6.05 90) (layer "F.Fab") hide
+    (fp_text value "ELQ3H7(TA)" (at 0 6.05 90) (layer "F.Fab") hide
       (effects (font (size 1 1) (thickness 0.15)))
     )
@@
     (fp_line (start -0.8 -0.4) (end 0.8 -0.4) (layer "F.Fab") (width 0.1))
     (pad "1" smd roundrect (at -0.775 0 180) (size 0.9 0.95) (layers "F.Cu" "F.Paste" "F.Mask") (roundrect_rratio 0.25)
-      (net 106 "Net-(U2-Pad5)") (pintype "passive"))
+      (net 106 "Net-(C6-Pad1)") (pintype "passive"))
     (pad "2" smd roundrect (at 0.775 0 180) (size 0.9 0.95) (layers "F.Cu" "F.Paste" "F.Mask") (roundrect_rratio 0.25)
-      (net 107 "Net-(U2-Pad6)") (pintype "passive"))
+      (net 107 "Net-(C6-Pad2)") (pintype "passive"))
     (model "${KICAD6_3DMODEL_DIR}/Capacitor_SMD.3dshapes/C_0603_1608Metric.wrl"
       (offset (xyz 0 0 0))
@@
   (segment (start 180.1927 89.5186) (end 180.1927 94.023427) (width 0.6096) (layer "F.Cu") (net 84))
   (segment (start 163.9315 88.519) (end 162.7854 89.6651) (width 0.6096) (layer "F.Cu") (net 84))
+  (segment (start 128.524 81.915) (end 127.635 82.804) (width 1.2192) (layer "F.Cu") (net 84))
   (segment (start 136.2759 94.023427) (end 137.16 94.907527) (width 0.6096) (layer "F.Cu") (net 84))
   (segment (start 168.2068 87.1514) (end 168.2068 88.519) (width 0.6096) (layer "F.Cu") (net 84))
@@
   (segment (start 177.038 87.249) (end 176.866 87.421) (width 0.6096) (layer "F.Cu") (net 84))
   (segment (start 127.5989 89.5111) (end 127.5989 94.023427) (width 0.6096) (layer "F.Cu") (net 84))
-  (segment (start 131.953 86.106) (end 131.953 84.201) (width 2.54) (layer "F.Cu") (net 84))
   (segment (start 144.952 70.56) (end 165.102 70.56) (width 2.54) (layer "F.Cu") (net 84))
   (segment (start 124.4345 88.519) (end 123.4079 89.5456) (width 0.6096) (layer "F.Cu") (net 84))
@@
   (segment (start 158.4749 89.5186) (end 158.4749 94.023427) (width 0.6096) (layer "F.Cu") (net 84))
   (segment (start 116.1995 88.519) (end 116.1995 87.6355) (width 0.6096) (layer "F.Cu") (net 84))
-  (segment (start 128.3385 82.423) (end 128.217 82.5445) (width 2.54) (layer "F.Cu") (net 84))
+  (segment (start 131.953 86.106) (end 130.683 84.836) (width 1.2192) (layer "F.Cu") (net 84))
   (segment (start 143.129 86.106) (end 159.258 86.106) (width 2.54) (layer "F.Cu") (net 84))
   (segment (start 175.8664 89.5186) (end 175.8664 94.023427) (width 0.6096) (layer "F.Cu") (net 84))
@@
   (segment (start 155.9204 87.1026) (end 155.3068 87.7162) (width 0.6096) (layer "F.Cu") (net 84))
   (segment (start 141.8335 88.519) (end 140.85005 89.50245) (width 0.6096) (layer "F.Cu") (net 84))
+  (segment (start 127.5265 82.804) (end 127.4314 82.7089) (width 1.2192) (layer "F.Cu") (net 84))
   (segment (start 176.866 88.519) (end 175.8664 89.5186) (width 0.6096) (layer "F.Cu") (net 84))
   (segment (start 150.9775 88.519) (end 149.9584 89.5381) (width 0.6096) (layer "F.Cu") (net 84))
@@
   (segment (start 150.9775 87.4015) (end 150.9775 88.519) (width 0.6096) (layer "F.Cu") (net 84))
   (segment (start 159.385 94.933527) (end 159.385 97.4439) (width 0.6096) (layer "F.Cu") (net 84))
+  (segment (start 127.635 82.804) (end 127.5265 82.804) (width 1.2192) (layer "F.Cu") (net 84))
   (segment (start 162.7854 94.023427) (end 163.576 94.814027) (width 0.6096) (layer "F.Cu") (net 84))
   (segment (start 159.258 86.106) (end 181.229 86.106) (width 2.54) (layer "F.Cu") (net 84))
@@
   (segment (start 172.548 87.548) (end 172.548 88.519) (width 0.6096) (layer "F.Cu") (net 84))
   (segment (start 127.5989 94.023427) (end 128.397 94.821527) (width 0.6096) (layer "F.Cu") (net 84))
-  (segment (start 130.175 82.423) (end 128.3385 82.423) (width 2.54) (layer "F.Cu") (net 84))
   (segment (start 159.4745 88.519) (end 158.4749 89.5186) (width 0.6096) (layer "F.Cu") (net 84))
   (segment (start 141.80485 94.978227) (end 141.80485 97.4482) (width 0.6096) (layer "F.Cu") (net 84))
@@
   (segment (start 128.591 87.309) (end 128.591 88.519) (width 0.6096) (layer "F.Cu") (net 84))
   (segment (start 168.021 97.3476) (end 168.1418 97.4684) (width 0.6096) (layer "F.Cu") (net 84))
-  (segment (start 131.953 84.201) (end 130.175 82.423) (width 2.54) (layer "F.Cu") (net 84))
+  (segment (start 130.683 84.836) (end 130.683 81.915) (width 1.2192) (layer "F.Cu") (net 84))
   (segment (start 171.5484 94.023427) (end 172.5032 94.978227) (width 0.6096) (layer "F.Cu") (net 84))
   (segment (start 176.784 94.941027) (end 176.784 97.4514) (width 0.6096) (layer "F.Cu") (net 84))
@@
   (segment (start 163.576 97.3244) (end 163.72 97.4684) (width 0.6096) (layer "F.Cu") (net 84))
   (segment (start 154.3072 94.023427) (end 155.262 94.978227) (width 0.6096) (layer "F.Cu") (net 84))
+  (segment (start 130.683 81.915) (end 128.524 81.915) (width 1.2192) (layer "F.Cu") (net 84))
   (segment (start 141.777 73.735) (end 144.952 70.56) (width 2.54) (layer "F.Cu") (net 84))
   (segment (start 149.9584 89.5381) (end 149.9584 94.023427) (width 0.6096) (layer "F.Cu") (net 84))
@@
   (segment (start 142.113 87.20885) (end 141.8335 87.48835) (width 0.6096) (layer "F.Cu") (net 84))
   (segment (start 120.015 97.2049) (end 120.015 94.694527) (width 0.6096) (layer "F.Cu") (net 84))
+  (segment (start 127.4314 82.7089) (end 127.4314 82.5445) (width 1.2192) (layer "F.Cu") (net 84))
   (segment (start 117.792 97.4684) (end 117.792 97.9885) (width 0.6096) (layer "F.Cu") (net 85))
   (segment (start 123.591 106.6925) (end 124.206 106.6925) (width 0.6096) (layer "F.Cu") (net 85))

Commit message: added 3d models
Parts:
- J3, J4: footprint Austins creations:2pinblock -> Vizista:CONN-TH_WJ2EDGVC-5.08-2P
- moved D2 32.1 mm to (150.9, 79.6)
- moved R1 32.0 mm to (150.6, 76.4)
- moved C7 30.9 mm to (154.4, 79.6)
- moved C9 30.9 mm to (161.6, 81.0)
- moved U2 30.9 mm to (158.2, 81.3)
- moved C8 30.9 mm to (154.4, 82.4)
- moved L1 30.9 mm to (158.1, 72.9)
- moved C6 30.9 mm to (158.3, 78.1)
- moved J3 20.4 mm to (119.9, 80.1), turned to -90 degrees
- moved J4 15.2 mm to (179.4, 80.5), turned to 90 degrees
- moved D3 11.5 mm to (164.8, 81.3)
- moved R5 11.0 mm to (167.8, 81.6)
- moved C5 10.8 mm to (142.0, 79.3), turned to 90 degrees
Routing:
- net VDD: track 300.9 -> 286.4 mm
- net +5V: track 121.4 -> 116.3 mm
- net GNDPWR: vias 23 -> 19

Commit message: clean up
Parts:
- moved D7 7.62 mm to (161.0, 50.8)
- moved RN7 5.24 mm to (126.4, 37.8)
- moved RN16 5.05 mm to (133.7, 37.7)
- moved RN12 4.62 mm to (133.7, 42.1)
- moved RN9 4.50 mm to (129.1, 42.0)
- moved RN5 4.04 mm to (154.1, 37.7)
- moved RN3 4.04 mm to (154.1, 42.2)
- moved R1 3.60 mm to (150.1, 80.0)
- moved D2 2.90 mm to (150.8, 82.4)
- moved R5 2.20 mm to (166.4, 79.9)
- moved C9 1.50 mm to (162.2, 82.4), turned to 180 degrees
- moved D3 1.41 mm to (165.8, 82.4)
- moved J1 0.87 mm to (179.9, 54.9)
- moved J3 0.44 mm to (119.9, 80.6)
- moved J4 0.17 mm to (179.4, 80.6)
Routing:
- net Net-(RN12-Pad8): track 7.81 -> 2.70 mm
- net Net-(RN12-Pad7): track 7.61 -> 2.51 mm
- net Net-(RN16-Pad6): track 7.66 -> 2.61 mm
- net Net-(RN16-Pad7): track 7.85 -> 2.81 mm
- net Net-(RN16-Pad5): track 7.46 -> 2.42 mm
- net Net-(RN12-Pad6): track 7.48 -> 2.49 mm
- net Net-(RN12-Pad5): track 7.67 -> 2.68 mm
- net Net-(RN16-Pad8): track 8.05 -> 3.10 mm
- net VDD: track 286.4 -> 281.5 mm
- net p3-c: track 36.7 -> 32.1 mm
- net p4-a: track 34.0 -> 29.6 mm
- net p3-a: track 26.6 -> 22.5 mm
- net p3-b: track 29.5 -> 25.4 mm
- net p4-d: track 38.5 -> 35.8 mm
- net p3-b5: track 28.5 -> 31.2 mm
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