File: RJ45toTerminal/RJ45-To-Terminal.kicad_sch (KiCad schematic)
At the start: 69 parts, among them J11 Screw_Terminal_01x08, J12 Screw_Terminal_01x08, J13 Screw_Terminal_01x08, J14 Screw_Terminal_01x08

Commit message: updated RJ45ToTerminal with additional space between pluggable conenctor
Parts:
- removed J11, J12, J13, J14: Screw_Terminal_01x08, VizistaHA:CONN-TH_4P-P3.50_JILN_JL15EDGRHC-35004B02, symbol Connector:Screw_Terminal_01x08
- added J11, J13, J16, J18: Screw_Terminal_01x04, Footprints:CONN-TH_XY2500V-F-3.5-4P, symbol Connector:Screw_Terminal_01x04
- added J12, J14, J17, J19: Screw_Terminal_01x04, Footprints:CONN-TH_XY2500R-G-3.5-4P, symbol Connector:Screw_Terminal_01x04
- D51, D52, D53, D54, D55, D56, D57, D58, D59, D60, D61, D62, D63, D64, D65, D66: LCSC C727080 -> C94470
- RJ45-1: LCSC C77852 -> C386760
Connections:
- net IN1-: now also J19.4 (Pin_4)
- net IN10-: now also J14.2 (Pin_2)
- net IN11-: now also J13.4 (Pin_4)
- net IN12-: now also J13.2 (Pin_2)
- net IN13-: now also J12.4 (Pin_4)
- net IN14-: now also J12.2 (Pin_2)
- net IN15-: now also J11.4 (Pin_4)
- net IN16-: now also J11.2 (Pin_2)
- net IN2-: now also J19.2 (Pin_2)
- net IN3-: now also J18.4 (Pin_4)
- net IN4-: now also J18.2 (Pin_2)
- net IN5-: now also J17.4 (Pin_4)
- net IN6-: now also J17.2 (Pin_2)
- net IN7-: now also J16.4 (Pin_4)
- net IN8-: now also J16.2 (Pin_2)
- net IN9-: now also J14.4 (Pin_4)
- net RC1-: now also J19.3 (Pin_3)
- net RC10-: now also J14.1 (Pin_1)
- net RC11-: now also J13.3 (Pin_3)
- net RC12-: now also J13.1 (Pin_1)
- net RC13-: now also J12.3 (Pin_3)
- net RC14-: now also J12.1 (Pin_1)
- net RC15-: now also J11.3 (Pin_3)
- net RC16-: now also J11.1 (Pin_1)
- net RC2-: now also J19.1 (Pin_1)
- net RC3-: now also J18.3 (Pin_3)
- net RC4-: now also J18.1 (Pin_1)
- net RC5-: now also J17.3 (Pin_3)
- net RC6-: now also J17.1 (Pin_1)
- net RC7-: now also J16.3 (Pin_3)
- net RC8-: now also J16.1 (Pin_1)
- net RC9-: now also J14.3 (Pin_3)

Commit message: 5V input suport
Parts:
- LED51, LED52, LED53, LED54, LED55, LED56, LED57, LED58, LED59, LED60, LED61, LED62, LED63, LED64, LED65, LED66: LCSC C72038 -> C2286; LCSC1 (none) -> C72038

Commit message: Fixed foot print and lcsc part id
Parts:
- RJ45-1: LCSC C386760 -> C77852
Changed lines of the file:
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@@
 			)
 		)
-		(property "LCSC" "C386760"
+		(property "LCSC" "C77852"
 			(at 54.61 48.26 0)
 			(effects

Commit message: fixes
Parts:
- added H1, H2, H3, H4, H5, H6: MountingHole, MountingHole:MountingHole_3.2mm_M3, symbol Mechanical:MountingHole
