File: rev 2/Modular-I2C-4PxRJ45-Relay-Driver.kicad_pcb (KiCad board)
At the start: 2 copper layers, 69.5 x 100 mm, 144 parts, among them J1 Conn_02x03_Odd_Even, J2 Conn_02x03_Odd_Even, J3 Screw_Terminal_01x02, J4 Screw_Terminal_01x02, Q51 2N7002, Q52 2N7002, Q53 2N7002, Q54 2N7002, Q55 2N7002, Q56 2N7002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

Commit message: Fixed foot print and lcsc part id
Parts:
- turned J4 to 90 degrees
Routing:
- net VDD: track 129.8 -> 138.7 mm
Changed lines of the file:
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@@
 	(footprint "Vizista:CONN-TH_WJ2EDGVC-5.08-2P"
 		(layer "F.Cu")
-		(at 179.3679 80.5688 -90)
+		(at 179.3679 80.5688 90)
 		(property "Reference" "J4"
 			(at -0.213 -4.608 90)
@@
 					(thickness 0.152)
 				)
-				(justify right)
+				(justify left)
 			)
 		)
@@
 					(thickness 0.152)
 				)
-				(justify right)
+				(justify left)
 			)
 		)
@@
 			)
 		)
-		(property "LCSC" "C3703"
+		(property "LCSC" "C8445"
 			(at 260.0027 -98.7331 0)
 			(layer "F.Fab")
@@
 		(attr through_hole)
 		(fp_line
-			(start -6.03 3.9)
-			(end -6.03 -4.191)
+			(start 6.096 -4.191)
+			(end 6.096 3.9)
 			(stroke
 				(width 0.254)
@@
 		)
 		(fp_line
-			(start 6.096 3.9)
-			(end -6.03 3.9)
+			(start -6.03 -4.191)
+			(end 6.096 -4.191)
 			(stroke
 				(width 0.254)
@@
 		)
 		(fp_line
-			(start -0.762 2.839)
-			(end 0.935 2.839)
+			(start 4.826 -2.794)
+			(end -4.699 -2.794)
 			(stroke
 				(width 0.254)
@@
 		)
 		(fp_line
-			(start 4.237 2.839)
-			(end 4.826 2.839)
+			(start -4.699 -2.794)
+			(end -4.699 2.794)
 			(stroke
 				(width 0.254)
@@
 		)
 		(fp_line
-			(start 4.826 2.839)
-			(end 4.826 -2.794)
+			(start -4.191 2.794)
+			(end -4.064 2.794)
 			(stroke
 				(width 0.254)
@@
 		)
 		(fp_line
-			(start -4.191 2.794)
-			(end -4.064 2.794)
+			(start 4.826 2.839)
+			(end 4.826 -2.794)
 			(stroke
 				(width 0.254)
@@
 		)
 		(fp_line
-			(start -4.699 -2.794)
-			(end -4.699 2.794)
+			(start 4.237 2.839)
+			(end 4.826 2.839)
 			(stroke
 				(width 0.254)
@@
 		)
 		(fp_line
-			(start 4.826 -2.794)
-			(end -4.699 -2.794)
+			(start -0.762 2.839)
+			(end 0.935 2.839)
 			(stroke
 				(width 0.254)
@@
 		)
 		(fp_line
-			(start -6.03 -4.191)
-			(end 6.096 -4.191)
+			(start 6.096 3.9)
+			(end -6.03 3.9)
 			(stroke
 				(width 0.254)
@@
 		)
 		(fp_line
-			(start 6.096 -4.191)
-			(end 6.096 3.9)
+			(start -6.03 3.9)
+			(end -6.03 -4.191)
 			(stroke
 				(width 0.254)
@@
 		)
 		(fp_arc
-			(start -0.762 2.839)
-			(mid -2.413056 3.601205)
-			(end -4.064073 2.838914)
+			(start 4.237 2.839)
+			(mid 2.585944 3.601205)
+			(end 0.934927 2.838914)
 			(stroke
 				(width 0.254)
@@
 		)
 		(fp_arc
-			(start 4.237 2.839)
-			(mid 2.585944 3.601205)
-			(end 0.934927 2.838914)
+			(start -0.762 2.839)
+			(mid -2.413056 3.601205)
+			(end -4.064073 2.838914)
 			(stroke
 				(width 0.254)
@@
 		)
 		(pad "1" thru_hole circle
-			(at -2.499 0 270)
+			(at -2.499 0 90)
 			(size 3 3)
 			(drill 1.7)
@@
 		)
 		(pad "2" thru_hole circle
-			(at 2.499 0 270)
+			(at 2.499 0 90)
 			(size 3 3)
 			(drill 1.7)
@@
 			)
 		)
-		(property "LCSC" "C3703"
+		(property "LCSC" "C8445"
 			(at 39.37 200.5076 0)
 			(layer "F.Fab")
@@
 	)
 	(gr_arc
-		(start 173.45 79.64)
-		(mid 173.096447 79.493553)
-		(end 172.95 79.14)
+		(start 173.45 84.8436)
+		(mid 173.096447 84.697153)
+		(end 172.95 84.3436)
 		(stroke
 			(width 0.15)
@@
 	)
 	(gr_line
-		(start 174.900047 76.649953)
-		(end 174.900047 79.149953)
+		(start 174.900047 81.853553)
+		(end 174.900047 84.353553)
 		(stroke
 			(width 0.15)
@@
 	)
 	(gr_line
-		(start 174.4 85.15)
-		(end 173.4 85.15)
+		(start 174.5 80)
+		(end 173.5 80)
 		(stroke
 			(width 0.15)
@@
 	)
 	(gr_arc
-		(start 174.400047 76.149953)
-		(mid 174.7536 76.2964)
-		(end 174.900047 76.649953)
+		(start 174.400047 81.353553)
+		(mid 174.7536 81.5)
+		(end 174.900047 81.853553)
 		(stroke
 			(width 0.15)
@@
 	)
 	(gr_arc
-		(start 174.9 84.65)
-		(mid 174.753553 85.003553)
-		(end 174.4 85.15)
+		(start 175 79.5)
+		(mid 174.853553 79.853553)
+		(end 174.5 80)
 		(stroke
 			(width 0.15)
@@
 	)
 	(gr_arc
-		(start 172.95 76.64)
-		(mid 173.096447 76.286447)
-		(end 173.45 76.14)
+		(start 172.95 81.8436)
+		(mid 173.096447 81.490047)
+		(end 173.45 81.3436)
 		(stroke
 			(width 0.15)
@@
 	)
 	(gr_arc
-		(start 173.4 85.15)
-		(mid 173.046447 85.003553)
-		(end 172.9 84.65)
+		(start 173.5 80)
+		(mid 173.146447 79.853553)
+		(end 173 79.5)
 		(stroke
 			(width 0.15)
@@
 	)
 	(gr_line
-		(start 172.95 79.14)
-		(end 172.95 76.64)
+		(start 172.95 84.3436)
+		(end 172.95 81.8436)
 		(stroke
 			(width 0.15)
@@
 	)
 	(gr_line
-		(start 172.9 84.65)
-		(end 172.9 82.15)
+		(start 173 79.5)
+		(end 173 77)
 		(stroke
 			(width 0.15)
@@
 	)
 	(gr_arc
-		(start 174.900047 79.149953)
-		(mid 174.7536 79.503506)
-		(end 174.400047 79.649953)
+		(start 174.900047 84.353553)
+		(mid 174.7536 84.707106)
+		(end 174.400047 84.853553)
 		(stroke
 			(width 0.15)
@@
 	)
 	(gr_arc
-		(start 172.9 82.15)
-		(mid 173.046447 81.796447)
-		(end 173.4 81.65)
+		(start 173 77)
+		(mid 173.146447 76.646447)
+		(end 173.5 76.5)
 		(stroke
 			(width 0.15)
@@
 	)
 	(gr_line
-		(start 174.4 81.65)
-		(end 173.4 81.65)
+		(start 174.5 76.5)
+		(end 173.5 76.5)
 		(stroke
 			(width 0.15)
@@
 	)
 	(gr_line
-		(start 174.400047 79.649953)
-		(end 173.45 79.639999)
+		(start 174.400047 84.853553)
+		(end 173.45 84.843599)
 		(stroke
 			(width 0.15)
@@
 	)
 	(gr_line
-		(start 173.350733 76.149953)
-		(end 174.400047 76.149953)
+		(start 173.350733 81.353553)
+		(end 174.400047 81.353553)
 		(stroke
 			(width 0.15)
@@
 	)
 	(gr_line
-		(start 174.9 84.65)
-		(end 174.9 82.15)
+		(start 175 79.5)
+		(end 175 77)
 		(stroke
 			(width 0.15)
@@
 	)
 	(gr_arc
-		(start 174.4 81.65)
-		(mid 174.753553 81.796447)
-		(end 174.9 82.15)
+		(start 174.5 76.5)
+		(mid 174.853553 76.646447)
+		(end 175 77)
 		(stroke
 			(width 0.15)
@@
 	)
 	(gr_text "GND"
-		(at 173.9 83.4 270)
+		(at 174 78.25 270)
 		(layer "F.SilkS")
 		(effects
@@
 	)
 	(gr_text "VIN"
-		(at 173.75 77.87 270)
+		(at 173.75 83.0736 270)
 		(layer "F.SilkS")
 		(effects
@@
 	)
 	(segment
-		(start 119.9388 78.0698)
-		(end 119.9388 68.453604)
+		(start 182.5 75.5)
+		(end 179.5 72.5)
+		(width 2.54)
+		(layer "F.Cu")
+		(net 84)
+	)
+	(segment
+		(start 126.428404 61.964)
+		(end 172.864 61.964)
 		(width 2.54)
 		(layer "F.Cu")
@@
 	)
 	(segment
-		(start 179.3679 68.6321)
-		(end 179.3679 78.0698)
-		(width 2.54)
-		(layer "F.Cu")
-		(net 84)
-	)
-	(segment
-		(start 172.864 61.964)
-		(end 179.45 68.55)
-		(width 2.54)
-		(layer "F.Cu")
-		(net 84)
-	)
-	(segment
 		(start 164.9625 79.975001)
 		(end 166.212501 78.725)
@@
 	)
 	(segment
-		(start 169.5 78.725)
-		(end 170.775 78.725)
-		(width 1.2192)
+		(start 172.864 61.964)
+		(end 179.5 68.6)
+		(width 2.54)
 		(layer "F.Cu")
 		(net 84)
@@
 	)
 	(segment
-		(start 126.428404 61.964)
-		(end 172.864 61.964)
+		(start 179.3679 83.0678)
+		(end 182.5 79.9357)
 		(width 2.54)
 		(layer "F.Cu")
@@
 	)
 	(segment
-		(start 179.45 68.55)
-		(end 179.3679 68.6321)
-		(width 2.54)
+		(start 169.5 78.725)
+		(end 175.0251 78.725)
+		(width 1.2192)
 		(layer "F.Cu")
 		(net 84)
 	)
 	(segment
-		(start 170.775 78.725)
-		(end 171.4302 78.0698)
+		(start 136.715 83)
+		(end 140 79.715)
 		(width 1.2192)
 		(layer "F.Cu")
@@
 	)
 	(segment
-		(start 136.715 83)
-		(end 140 79.715)
-		(width 1.2192)
+		(start 119.9388 78.0698)
+		(end 119.9388 68.453604)
+		(width 2.54)
 		(layer "F.Cu")
 		(net 84)
@@
 	)
 	(segment
+		(start 179.5 72.5)
+		(end 179.5 68.7642)
+		(width 2.54)
+		(layer "F.Cu")
+		(net 84)
+	)
+	(segment
 		(start 164.9625 80.45)
 		(end 164.9625 79.975001)
@@
 	)
 	(segment
-		(start 140.015 79.73)
-		(end 140 79.715)
+		(start 175.0251 78.725)
+		(end 179.3679 83.0678)
 		(width 1.2192)
 		(layer "F.Cu")
@@
 	)
 	(segment
-		(start 171.4302 78.0698)
-		(end 179.3679 78.0698)
+		(start 182.5 79.9357)
+		(end 182.5 75.5)
+		(width 2.54)
+		(layer "F.Cu")
+		(net 84)
+	)
+	(segment
+		(start 140.015 79.73)
+		(end 140 79.715)
 		(width 1.2192)
 		(layer "F.Cu")

Commit message: fixes
Parts:
- J3, J4: footprint Vizista:CONN-TH_WJ2EDGVC-5.08-2P -> LCSC:LCSC-C8465-CONN-TH_2P-P5.00_WJ500V-5.08-2P
- moved J4 1.27 mm to (178.5, 81.5), turned to 0 degrees
- moved J3 1.09 mm to (120.5, 81.5), turned to 0 degrees
- moved R5 0.25 mm to (165.8, 82.2)
Routing:
- net VDD: track 138.7 -> 140.8 mm
Other:
- board text added: "J3"
- board text added: "J4"
- board text removed: "VIN 12v"
