File: rev 2/Modular-I2C-4PxRJ45-Relay-Driver.kicad_sch (KiCad schematic)
At the start: 123 parts, among them J1 Conn_02x03_Odd_Even, J2 Conn_02x03_Odd_Even, J3 Screw_Terminal_01x02, J4 Screw_Terminal_01x02, Q51 2N7002, Q52 2N7002, Q53 2N7002, Q54 2N7002, Q55 2N7002, Q56 2N7002, Q57 2N7002, Q58 2N7002, Q59 2N7002, Q60 2N7002, Q61 2N7002, Q62 2N7002, Q63 2N7002, Q64 2N7002, Q65 2N7002, Q66 2N7002, SW1 SW_DIP_x04, SW5 2P_DIP, U1 MCP23017_SO, U2 AP63205WU, U3 ELQ3H7(TA), U4 ELQ3H7(TA), U5 ELQ3H7(TA), U6 ELQ3H7(TA)

Commit message: updated RJ45ToTerminal with additional space between pluggable conenctor
Parts:
- D51: LCSC C727080 -> C94470; LCSC_old (none) -> C727080
- D52, D53, D54, D55, D56, D57, D58, D59, D60, D61, D62, D63, D64, D65, D66: LCSC C727080 -> C94470
Changed lines of the file:
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@@
       (effects (font (size 1.27 1.27)) hide)
     )
-    (property "LCSC" "C727080" (id 4) (at 360.68 -55.88 90)
+    (property "LCSC" "C94470" (id 4) (at 360.68 -55.88 90)
       (effects (font (size 1 1)))
     )
@@
       (effects (font (size 1.27 1.27)) hide)
     )
-    (property "LCSC" "C727080" (id 4) (at -109.22 45.72 90)
+    (property "LCSC_old" "C727080" (id 4) (at -109.22 45.72 90)
+      (effects (font (size 1 1)) hide)
+    )
+    (property "LCSC" "C94470" (id 5) (at -115.57 44.45 90)
       (effects (font (size 1 1)))
     )
@@
       (effects (font (size 1.27 1.27)) hide)
     )
-    (property "LCSC" "C727080" (id 4) (at 360.68 -139.7 90)
+    (property "LCSC" "C94470" (id 4) (at 360.68 -139.7 90)
       (effects (font (size 1 1)))
     )
@@
       (effects (font (size 1.27 1.27)) hide)
     )
-    (property "LCSC" "C727080" (id 4) (at 227.33 -140.97 90)
+    (property "LCSC" "C94470" (id 4) (at 227.33 -140.97 90)
       (effects (font (size 1 1)))
     )
@@
       (effects (font (size 1.27 1.27)) hide)
     )
-    (property "LCSC" "C727080" (id 4) (at 227.33 -57.15 90)
+    (property "LCSC" "C94470" (id 4) (at 227.33 -57.15 90)
       (effects (font (size 1 1)))
     )
@@
       (effects (font (size 1.27 1.27)) hide)
     )
-    (property "LCSC" "C727080" (id 4) (at 227.33 -113.03 90)
+    (property "LCSC" "C94470" (id 4) (at 227.33 -113.03 90)
       (effects (font (size 1 1)))
     )
@@
       (effects (font (size 1.27 1.27)) hide)
     )
-    (property "LCSC" "C727080" (id 4) (at -109.22 130.81 90)
+    (property "LCSC" "C94470" (id 4) (at -109.22 130.81 90)
       (effects (font (size 1 1)))
     )
@@
       (effects (font (size 1.27 1.27)) hide)
     )
-    (property "LCSC" "C727080" (id 4) (at 97.79 -111.76 90)
+    (property "LCSC" "C94470" (id 4) (at 97.79 -111.76 90)
       (effects (font (size 1 1)))
     )
@@
       (effects (font (size 1.27 1.27)) hide)
     )
-    (property "LCSC" "C727080" (id 4) (at 227.33 -85.09 90)
+    (property "LCSC" "C94470" (id 4) (at 227.33 -85.09 90)
       (effects (font (size 1 1)))
     )
@@
       (effects (font (size 1.27 1.27)) hide)
     )
-    (property "LCSC" "C727080" (id 4) (at -109.22 74.93 90)
+    (property "LCSC" "C94470" (id 4) (at -109.22 74.93 90)
       (effects (font (size 1 1)))
     )
@@
       (effects (font (size 1.27 1.27)) hide)
     )
-    (property "LCSC" "C727080" (id 4) (at 97.79 -55.88 90)
+    (property "LCSC" "C94470" (id 4) (at 97.79 -55.88 90)
       (effects (font (size 1 1)))
     )
@@
       (effects (font (size 1.27 1.27)) hide)
     )
-    (property "LCSC" "C727080" (id 4) (at 360.68 -83.82 90)
+    (property "LCSC" "C94470" (id 4) (at 360.68 -83.82 90)
       (effects (font (size 1 1)))
     )
@@
       (effects (font (size 1.27 1.27)) hide)
     )
-    (property "LCSC" "C727080" (id 4) (at -109.22 102.87 90)
+    (property "LCSC" "C94470" (id 4) (at -109.22 102.87 90)
       (effects (font (size 1 1)))
     )
@@
       (effects (font (size 1.27 1.27)) hide)
     )
-    (property "LCSC" "C727080" (id 4) (at 360.68 -111.76 90)
+    (property "LCSC" "C94470" (id 4) (at 360.68 -111.76 90)
       (effects (font (size 1 1)))
     )
@@
       (effects (font (size 1.27 1.27)) hide)
     )
-    (property "LCSC" "C727080" (id 4) (at 97.79 -83.82 90)
+    (property "LCSC" "C94470" (id 4) (at 97.79 -83.82 90)
       (effects (font (size 1 1)))
     )
@@
       (effects (font (size 1.27 1.27)) hide)
     )
-    (property "LCSC" "C727080" (id 4) (at 97.79 -139.7 90)
+    (property "LCSC" "C94470" (id 4) (at 97.79 -139.7 90)
       (effects (font (size 1 1)))
     )

Commit message: updated to support 5V output for fan speed control in rev2
Parts:
- added D67, D68, D69, D70, D71, D72, D73, D74, D75, D76, D77, D78, D79, D80, D81, D82: 1N4004 SMB, LCSC:LCSC-C94470-MICROSMP_L2.2-W1.3-LS2.5-RD, symbol Diode:1N4004
- added JP1: Jumper_3_Open, Connector_PinHeader_2.54mm:PinHeader_1x03_P2.54mm_Vertical, symbol Jumper:Jumper_3_Open
Connections:
- net +5V: now also JP1.1 (A)
- net VDD: now also JP1.3 (B); no longer LED51.2 (A), LED52.2 (A), LED53.2 (A), LED54.2 (A), LED55.2 (A), LED56.2 (A), LED57.2 (A), LED58.2 (A), LED59.2 (A), LED60.2 (A), LED61.2 (A), LED62.2 (A), LED63.2 (A), LED64.2 (A), LED65.2 (A), LED66.2 (A), TH51.1, TH52.1, TH53.1, TH54.1, TH55.1, TH56.1, TH57.1, TH58.1, TH59.1, TH60.1, TH61.1, TH62.1, TH63.1, TH64.1, TH65.1, TH66.1
- net p1-a5: now also D70.1 (K); no longer U3.9 (Pin_9)
- net p1-b5: now also D69.1 (K); no longer U3.11 (Pin_11)
- net p1-c5: now also D68.1 (K); no longer U3.13 (Pin_13)
- net p1-d5: now also D67.1 (K); no longer U3.15 (Pin_15)
- net p2-a5: now also D71.1 (K); no longer U4.9 (Pin_9)
- net p2-b5: now also D72.1 (K); no longer U4.11 (Pin_11)
- net p2-c5: now also D73.1 (K); no longer U4.13 (Pin_13)
- net p2-d5: now also D74.1 (K); no longer U4.15 (Pin_15)
- net p3-a5: now also D75.1 (K); no longer U5.9 (Pin_9)
- net p3-b5: now also D76.1 (K); no longer U5.11 (Pin_11)
- net p3-c5: now also D77.1 (K); no longer U5.13 (Pin_13)
- net p3-d5: now also D78.1 (K); no longer U5.15 (Pin_15)
- net p4-a5: now also D79.1 (K); no longer U6.9 (Pin_9)
- net p4-b5: now also D80.1 (K); no longer U6.11 (Pin_11)
- net p4-c5: now also D81.1 (K); no longer U6.13 (Pin_13)
- net p4-d5: now also D82.1 (K); no longer U6.15 (Pin_15)
- new net: D69.2 (A), U3.11 (Pin_11)
- new net: D72.2 (A), U4.11 (Pin_11)
- new net: D73.2 (A), U4.13 (Pin_13)
- new net: D74.2 (A), U4.15 (Pin_15)
- new net: D71.2 (A), U4.9 (Pin_9)
- new net: D79.2 (A), U6.9 (Pin_9)
- new net: D78.2 (A), U5.15 (Pin_15)
- new net: D76.2 (A), U5.11 (Pin_11)
- new net: D67.2 (A), U3.15 (Pin_15)
- new net: D75.2 (A), U5.9 (Pin_9)
- new net: D68.2 (A), U3.13 (Pin_13)
- new net: D70.2 (A), U3.9 (Pin_9)
- new net: D77.2 (A), U5.13 (Pin_13)
- new net: D81.2 (A), U6.13 (Pin_13)
- new net: D80.2 (A), U6.11 (Pin_11)
- new net: D82.2 (A), U6.15 (Pin_15)
- new net ADJV: JP1.2 (C), LED51.2 (A), LED52.2 (A), LED53.2 (A), LED54.2 (A), LED55.2 (A), LED56.2 (A), LED57.2 (A), LED58.2 (A), LED59.2 (A), LED60.2 (A), LED61.2 (A), LED62.2 (A), LED63.2 (A), LED64.2 (A), LED65.2 (A), LED66.2 (A), TH51.1, TH52.1, TH53.1, TH54.1, TH55.1, TH56.1, TH57.1, TH58.1, TH59.1, TH60.1, TH61.1, TH62.1, TH63.1, TH64.1, TH65.1, TH66.1
Other:
- moved on the sheet: C1, C3, C5, D1, D3, D4, D5, D51, D52, D53, D54, D6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

Commit message: 5V input suport
Parts:
- added JP2: Jumper_3_Open, Connector_PinHeader_2.54mm:PinHeader_1x03_P2.54mm_Vertical, symbol Jumper:Jumper_3_Open
- added JP3: Jumper_2_Small_Open, Connector_PinHeader_2.54mm:PinHeader_1x02_P2.54mm_Vertical, symbol Jumper:Jumper_2_Small_Open
- C7, C8: LCSC C19702 -> C84419
- D2, D3, LED51, LED52, LED53, LED54, LED55, LED56, LED57, LED58, LED59, LED60, LED61, LED62, LED63, LED64, LED65, LED66: LCSC C72038 -> C2286
- Q51, Q52, Q53, Q54, Q55, Q56, Q57, Q58, Q59, Q60, Q61, Q62, Q63, Q64, Q65, Q66: LCSC C526325 -> C8545
Connections:
- net +5V: now also JP2.1 (A); no longer U3.10 (Pin_10), U3.12 (Pin_12), U3.14 (Pin_14), U3.16 (Pin_16), U4.10 (Pin_10), U4.12 (Pin_12), U4.14 (Pin_14), U4.16 (Pin_16), U5.10 (Pin_10), U5.12 (Pin_12), U5.14 (Pin_14), U5.16 (Pin_16), U6.10 (Pin_10), U6.12 (Pin_12), U6.14 (Pin_14), U6.16 (Pin_16)
- net VDD: now also JP2.3 (B), JP3.1 (A); no longer C9.2, U2.2 (EN), U2.3 (IN)
- new net 12VIN: C9.2, JP3.2 (B), U2.2 (EN), U2.3 (IN)
- new net OptoIN: JP2.2 (C), U3.10 (Pin_10), U3.12 (Pin_12), U3.14 (Pin_14), U3.16 (Pin_16), U4.10 (Pin_10), U4.12 (Pin_12), U4.14 (Pin_14), U4.16 (Pin_16), U5.10 (Pin_10), U5.12 (Pin_12), U5.14 (Pin_14), U5.16 (Pin_16), U6.10 (Pin_10), U6.12 (Pin_12), U6.14 (Pin_14), U6.16 (Pin_16)

Commit message: Fixed foot print and lcsc part id
Parts:
- J3, J4: LCSC C3703 -> C8445
Changed lines of the file:
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@@
 			)
 		)
-		(property "LCSC" "C3703"
+		(property "LCSC" "C8445"
 			(at 74.93 134.6199 0)
 			(effects
@@
 			)
 		)
-		(property "LCSC" "C3703"
+		(property "LCSC" "C8445"
 			(at 74.93 119.3799 0)
 			(effects

Commit message: fixes
Parts:
- J3, J4: footprint Vizista:CONN-TH_WJ2EDGVC-5.08-2P -> LCSC:LCSC-C8465-CONN-TH_2P-P5.00_WJ500V-5.08-2P; LCSC C8445 -> C8465
- SW1: LCSC C2758183 -> C129080; LCSC1 (none) -> C2758183
- SW5: LCSC C976364 -> C129078; LCSC1 (none) -> C976364
Changed lines of the file:
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@@
 			)
 		)
-		(property "LCSC" "C976364"
+		(property "LCSC" "C129078"
 			(at 118.11 137.16 0)
 			(effects
@@
 					(size 1.27 1.27)
 				)
+			)
+		)
+		(property "LCSC1" "C976364"
+			(at 118.11 142.24 0)
+			(effects
+				(font
+					(size 1 1)
+				)
+				(hide yes)
 			)
 		)
@@
 			)
 		)
-		(property "Footprint" "Vizista:CONN-TH_WJ2EDGVC-5.08-2P"
+		(property "Footprint" "LCSC:LCSC-C8465-CONN-TH_2P-P5.00_WJ500V-5.08-2P"
 			(at 69.85 127 0)
 			(effects
@@
 			)
 		)
-		(property "LCSC" "C8445"
+		(property "LCSC" "C8465"
 			(at 74.93 134.6199 0)
 			(effects
@@
 			)
 		)
-		(property "LCSC" "C2758183"
+		(property "LCSC" "C129080"
 			(at 40.64 82.55 0)
 			(effects
@@
 					(size 1.27 1.27)
 				)
+			)
+		)
+		(property "LCSC1" "C2758183"
+			(at 40.64 74.93 0)
+			(effects
+				(font
+					(size 1 1)
+				)
+				(hide yes)
 			)
 		)
@@
 			)
 		)
-		(property "Footprint" "Vizista:CONN-TH_WJ2EDGVC-5.08-2P"
+		(property "Footprint" "LCSC:LCSC-C8465-CONN-TH_2P-P5.00_WJ500V-5.08-2P"
 			(at 69.85 111.76 0)
 			(effects
@@
 			)
 		)
-		(property "LCSC" "C8445"
+		(property "LCSC" "C8465"
 			(at 74.93 119.3799 0)
 			(effects

Commit message: fixes
Parts:
- JP3: LCSC (none) -> C492401
Changed lines of the file:
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@@
+			)
+		)
+		(property "LCSC" "C492401"
+			(at 139.7 199.39 0)
+			(effects
+				(font
+					(size 1 1)
+				)
+				(hide yes)
 			)
 		)
